Commit message: SITL Gimbal xacro file added

File: urdf/macro_gimbal_3d.xacro (robot description, xacro)
@@ -5,20 +5,20 @@
     <xacro:property name="pi" value="3.141592653589793" />
     <xacro:property name="use_sim_time" value="true" />
-    <xacro:property name="gimbal_namespace" value="${namespace}_gimbal" />
+    <xacro:property name="namespace_gimbal" value="${namespace}_gimbal" />
     <xacro:property name="STREAM_PORT" value="${5600 + int(instance) * 10}" />
-    <link name="${gimbal_namespace}_base_link">
+    <link name="${namespace_gimbal}_base_link">
       <inertial>
         <mass value="0.2" />
         <inertia ixx="0.0001" ixy="0" ixz="0" iyy="0.0001" iyz="0" izz="0.0001" />
       </inertial>
-      <visual name="${gimbal_namespace}_base_visual">
+      <visual name="${namespace_gimbal}_base_visual">
         <geometry>
           <mesh filename="package://${package_name}/meshes/gimbal_3d/base_plate.dae" />
         </geometry>
-        <material name="${gimbal_namespace}_material">
+        <material name="${namespace_gimbal}_material">
           <color rgba="${rgb} 1" />
         </material>
       </visual>
-      <collision name="${gimbal_namespace}_base_collision">
+      <collision name="${namespace_gimbal}_base_collision">
         <origin xyz="0.01 0.075 -0.025" rpy="0 0 0" />
         <geometry>
@@ -27,16 +27,16 @@
       </collision>
     </link>
-    <gazebo reference="${gimbal_namespace}_base_link">
-      <visual name="${gimbal_namespace}_base_visual">
-        <material name="${gimbal_namespace}_material">
-          <diffuse>${rgb} 1</diffuse>
-          <ambient>${rgb} 1</ambient>
-          <specular>1 1 1 1</specular>
-        </material>
-      </visual>
-    </gazebo>
-    <joint name="${gimbal_namespace}_base_joint" type="fixed">
+    <gazebo reference="${namespace_gimbal}_base_link">
+      <visual name="${namespace_gimbal}_base_visual">
+        <material name="${namespace_gimbal}_material">
+          <diffuse>${rgb} 1</diffuse>
+          <ambient>${rgb} 1</ambient>
+          <specular>1 1 1 1</specular>
+        </material>
+      </visual>
+    </gazebo>
+    <joint name="${namespace_gimbal}_base_joint" type="fixed">
       <parent link="${parent_link}" />
-      <child link="${gimbal_namespace}_base_link" />
+      <child link="${namespace_gimbal}_base_link" />
       <origin xyz="${xyz}" rpy="${rpy}" />
       <axis xyz="0 0 1">
@@ -44,16 +44,16 @@
       </axis>
     </joint>
-    <link name="${gimbal_namespace}_yaw_link">
+    <link name="${namespace_gimbal}_yaw_link">
       <inertial>
         <mass value="0.01" />
         <inertia ixx="0.00001" ixy="0" ixz="0" iyy="0.00001" iyz="0" izz="0.00001" />
       </inertial>
-      <visual name="${gimbal_namespace}_yaw_visual">
+      <visual name="${namespace_gimbal}_yaw_visual">
         <geometry>
           <mesh filename="package://${package_name}/meshes/gimbal_3d/yaw_arm.dae" />
         </geometry>
-        <material name="${gimbal_namespace}_material" />
-      </visual>
-      <collision name="${gimbal_namespace}_yaw_collision">
+        <material name="${namespace_gimbal}_material" />
+      </visual>
+      <collision name="${namespace_gimbal}_yaw_collision">
         <geometry>
           <mesh filename="package://${package_name}/meshes/gimbal_3d/yaw_arm.dae" />
@@ -61,16 +61,16 @@
       </collision>
     </link>
-    <gazebo reference="${gimbal_namespace}_yaw_link">
-      <visual name="${gimbal_namespace}_yaw_visual">
-        <material name="${gimbal_namespace}_material">
-          <diffuse>${rgb} 1</diffuse>
-          <ambient>${rgb} 1</ambient>
-          <specular>1 1 1 1</specular>
-        </material>
-      </visual>
-    </gazebo>
-    <joint name="${gimbal_namespace}_yaw_joint" type="revolute">
-      <parent link="${gimbal_namespace}_base_link" />
-      <child link="${gimbal_namespace}_yaw_link" />
+    <gazebo reference="${namespace_gimbal}_yaw_link">
+      <visual name="${namespace_gimbal}_yaw_visual">
+        <material name="${namespace_gimbal}_material">
+          <diffuse>${rgb} 1</diffuse>
+          <ambient>${rgb} 1</ambient>
+          <specular>1 1 1 1</specular>
+        </material>
+      </visual>
+    </gazebo>
+    <joint name="${namespace_gimbal}_yaw_joint" type="revolute">
+      <parent link="${namespace_gimbal}_base_link" />
+      <child link="${namespace_gimbal}_yaw_link" />
       <origin xyz="0 0 0" rpy="0 0 0" />
       <axis xyz="0 1 0" />
@@ -78,16 +78,16 @@
       <dynamics damping="0.01" />
     </joint>
-    <link name="${gimbal_namespace}_roll_link">
+    <link name="${namespace_gimbal}_roll_link">
       <inertial>
         <mass value="0.01" />
         <inertia ixx="0.00001" ixy="0" ixz="0" iyy="0.00001" iyz="0" izz="0.00001" />
       </inertial>
-      <visual name="${gimbal_namespace}_roll_visual">
+      <visual name="${namespace_gimbal}_roll_visual">
         <geometry>
           <mesh filename="package://${package_name}/meshes/gimbal_3d/roll_arm.dae" />
         </geometry>
-        <material name="${gimbal_namespace}_material" />
-      </visual>
-      <collision name="${gimbal_namespace}_roll_collision">
+        <material name="${namespace_gimbal}_material" />
+      </visual>
+      <collision name="${namespace_gimbal}_roll_collision">
         <geometry>
           <mesh filename="package://${package_name}/meshes/gimbal_3d/roll_arm.dae" />
@@ -95,16 +95,16 @@
       </collision>
     </link>
-    <gazebo reference="${gimbal_namespace}_roll_link">
-      <visual name="${gimbal_namespace}_roll_visual">
-        <material name="${gimbal_namespace}_material">
-          <diffuse>${rgb} 1</diffuse>
-          <ambient>${rgb} 1</ambient>
-          <specular>1 1 1 1</specular>
-        </material>
-      </visual>
-    </gazebo>
-    <joint name="${gimbal_namespace}_roll_joint" type="revolute">
-      <parent link="${gimbal_namespace}_yaw_link" />
-      <child link="${gimbal_namespace}_roll_link" />
+    <gazebo reference="${namespace_gimbal}_roll_link">
+      <visual name="${namespace_gimbal}_roll_visual">
+        <material name="${namespace_gimbal}_material">
+          <diffuse>${rgb} 1</diffuse>
+          <ambient>${rgb} 1</ambient>
+          <specular>1 1 1 1</specular>
+        </material>
+      </visual>
+    </gazebo>
+    <joint name="${namespace_gimbal}_roll_joint" type="revolute">
+      <parent link="${namespace_gimbal}_yaw_link" />
+      <child link="${namespace_gimbal}_roll_link" />
       <origin xyz="0 0 0" rpy="0 0 0" />
       <axis xyz="0 0 1" />
@@ -112,28 +112,28 @@
       <dynamics damping="0.01" />
     </joint>
-    <link name="${gimbal_namespace}_pitch_link">
+    <link name="${namespace_gimbal}_pitch_link">
       <inertial>
         <mass value="0.01" />
         <inertia ixx="0.00001" ixy="0" ixz="0" iyy="0.00001" iyz="0" izz="0.00001" />
       </inertial>
-      <visual name="${gimbal_namespace}_camera_enclosure_visual">
+      <visual name="${namespace_gimbal}_camera_enclosure_visual">
         <geometry>
           <mesh filename="package://${package_name}/meshes/gimbal_3d/camera_enclosure.dae" />
         </geometry>
-        <material name="${gimbal_namespace}_material" />
-      </visual>
-      <collision name="${gimbal_namespace}_camera_enclosure_collision">
+        <material name="${namespace_gimbal}_material" />
+      </visual>
+      <collision name="${namespace_gimbal}_camera_enclosure_collision">
         <geometry>
           <mesh filename="package://${package_name}/meshes/gimbal_3d/camera_enclosure.dae" />
         </geometry>
       </collision>
-      <visual name="${gimbal_namespace}_camera_body_visual">
+      <visual name="${namespace_gimbal}_camera_body_visual">
         <origin xyz="0 0 0.02" rpy="0 0 0" />
         <geometry>
           <cylinder radius="0.025" length="0.050" />
         </geometry>
-        <material name="${gimbal_namespace}_material" />
-      </visual>
-      <collision name="${gimbal_namespace}_camera_body_collision">
+        <material name="${namespace_gimbal}_material" />
+      </visual>
+      <collision name="${namespace_gimbal}_camera_body_collision">
         <origin xyz="0 0 0.02" rpy="0 0 0" />
         <geometry>
@@ -142,23 +142,23 @@
       </collision>
     </link>
-    <gazebo reference="${gimbal_namespace}_pitch_link">
-      <visual name="${gimbal_namespace}_camera_enclosure_visual">
-        <material name="${gimbal_namespace}_material">
-          <diffuse>${rgb} 1</diffuse>
-          <ambient>${rgb} 1</ambient>
-          <specular>1 1 1 1</specular>
-        </material>
-      </visual>
-      <visual name="${gimbal_namespace}_camera_body_visual">
-        <material name="${gimbal_namespace}_material">
-          <diffuse>${rgb} 1</diffuse>
-          <ambient>${rgb} 1</ambient>
-          <specular>1 1 1 1</specular>
-        </material>
-      </visual>
-    </gazebo>
-    <joint name="${gimbal_namespace}_pitch_joint" type="revolute">
-      <parent link="${gimbal_namespace}_roll_link" />
-      <child link="${gimbal_namespace}_pitch_link" />
+    <gazebo reference="${namespace_gimbal}_pitch_link">
+      <visual name="${namespace_gimbal}_camera_enclosure_visual">
+        <material name="${namespace_gimbal}_material">
+          <diffuse>${rgb} 1</diffuse>
+          <ambient>${rgb} 1</ambient>
+          <specular>1 1 1 1</specular>
+        </material>
+      </visual>
+      <visual name="${namespace_gimbal}_camera_body_visual">
+        <material name="${namespace_gimbal}_material">
+          <diffuse>${rgb} 1</diffuse>
+          <ambient>${rgb} 1</ambient>
+          <specular>1 1 1 1</specular>
+        </material>
+      </visual>
+    </gazebo>
+    <joint name="${namespace_gimbal}_pitch_joint" type="revolute">
+      <parent link="${namespace_gimbal}_roll_link" />
+      <child link="${namespace_gimbal}_pitch_link" />
       <origin xyz="0 0 0" rpy="0 0 0" />
       <axis xyz="1 0 0" />
@@ -166,6 +166,6 @@
       <dynamics damping="0.01" />
     </joint>
-    <gazebo reference="${gimbal_namespace}_pitch_link">
-      <sensor name="${gimbal_namespace}_camera_sensor" type="camera">
+    <gazebo reference="${namespace_gimbal}_pitch_link">
+      <sensor name="${namespace_gimbal}_camera_sensor" type="camera">
         <pose>0 0 0 ${- pi / 2} ${- pi / 2} 0</pose>
         <camera>

File: urdf/macro_sitl_core.xacro (robot description, xacro)
@@ -2,8 +2,8 @@
 <robot xmlns:xacro="http://www.ros.org/wiki/xacro">
   <xacro:macro name="macro_sitl_core"
-    params="package_name:='fpv_drone' namespace:='fpv_drone' instance:='0'">
+    params="namespace:='fpv_drone' instance:='0'">
     <xacro:property name="SITL_PORT" value="${9002 + int(instance) * 10}" />
     <gazebo>
-      <xacro:macro name="liftdrag_plugin_macro" params="motor_prefix cp_vec fwd_vec">
+      <xacro:macro name="macro_liftdrag_plugin" params="motor_prefix cp_vec fwd_vec">
         <plugin filename="gz-sim-lift-drag-system" name="gz::sim::systems::LiftDrag">
           <link_name>${namespace}_motor_${motor_prefix}_link</link_name>
@@ -23,27 +23,27 @@
         </plugin>
       </xacro:macro>
-      <xacro:liftdrag_plugin_macro motor_prefix="fr" cp_vec="0.084 0 0"
+      <xacro:macro_liftdrag_plugin motor_prefix="fr" cp_vec="0.084 0 0"
         fwd_vec="0 1 0" />
-      <xacro:liftdrag_plugin_macro motor_prefix="fr" cp_vec="-0.042 0.0727 0"
+      <xacro:macro_liftdrag_plugin motor_prefix="fr" cp_vec="-0.042 0.0727 0"
         fwd_vec="-0.866 -0.5 0" />
-      <xacro:liftdrag_plugin_macro motor_prefix="fr" cp_vec="-0.042 -0.0727 0"
+      <xacro:macro_liftdrag_plugin motor_prefix="fr" cp_vec="-0.042 -0.0727 0"
         fwd_vec="0.866 -0.5 0" />
-      <xacro:liftdrag_plugin_macro motor_prefix="bl" cp_vec="0.084 0 0"
+      <xacro:macro_liftdrag_plugin motor_prefix="bl" cp_vec="0.084 0 0"
         fwd_vec="0 1 0" />
-      <xacro:liftdrag_plugin_macro motor_prefix="bl" cp_vec="-0.042 0.0727 0"
+      <xacro:macro_liftdrag_plugin motor_prefix="bl" cp_vec="-0.042 0.0727 0"
         fwd_vec="-0.866 -0.5 0" />
-      <xacro:liftdrag_plugin_macro motor_prefix="bl" cp_vec="-0.042 -0.0727 0"
+      <xacro:macro_liftdrag_plugin motor_prefix="bl" cp_vec="-0.042 -0.0727 0"
         fwd_vec="0.866 -0.5 0" />
-      <xacro:liftdrag_plugin_macro motor_prefix="fl" cp_vec="0.084 0 0"
+      <xacro:macro_liftdrag_plugin motor_prefix="fl" cp_vec="0.084 0 0"
         fwd_vec="0 -1 0" />
-      <xacro:liftdrag_plugin_macro motor_prefix="fl" cp_vec="-0.042 0.0727 0"
+      <xacro:macro_liftdrag_plugin motor_prefix="fl" cp_vec="-0.042 0.0727 0"
         fwd_vec="0.866 0.5 0" />
-      <xacro:liftdrag_plugin_macro motor_prefix="fl" cp_vec="-0.042 -0.0727 0"
+      <xacro:macro_liftdrag_plugin motor_prefix="fl" cp_vec="-0.042 -0.0727 0"
         fwd_vec="-0.866 0.5 0" />
-      <xacro:liftdrag_plugin_macro motor_prefix="br" cp_vec="0.084 0 0"
+      <xacro:macro_liftdrag_plugin motor_prefix="br" cp_vec="0.084 0 0"
         fwd_vec="0 -1 0" />
-      <xacro:liftdrag_plugin_macro motor_prefix="br" cp_vec="-0.042 0.0727 0"
+      <xacro:macro_liftdrag_plugin motor_prefix="br" cp_vec="-0.042 0.0727 0"
         fwd_vec="0.866 0.5 0" />
-      <xacro:liftdrag_plugin_macro motor_prefix="br" cp_vec="-0.042 -0.0727 0"
+      <xacro:macro_liftdrag_plugin motor_prefix="br" cp_vec="-0.042 -0.0727 0"
         fwd_vec="-0.866 0.5 0" />
       <xacro:macro name="apply_joint_force_plugin_macro" params="motor_prefix">
@@ -66,5 +66,5 @@
         <gazeboXYZToNED degrees="true">0 0 0 180 0 90</gazeboXYZToNED>
         <imuName>${namespace}_imu_link::${namespace}_imu_sensor</imuName>
-        <xacro:macro name="control_motor_macro" params="channel motor_prefix multiplier">
+        <xacro:macro name="macro_control_motor" params="channel motor_prefix multiplier">
           <control channel="${channel}">
             <jointName>${namespace}_motor_${motor_prefix}_joint</jointName>
@@ -85,8 +85,8 @@
           </control>
         </xacro:macro>
-        <xacro:control_motor_macro channel="0" motor_prefix="fr" multiplier="838" />
-        <xacro:control_motor_macro channel="1" motor_prefix="bl" multiplier="838" />
-        <xacro:control_motor_macro channel="2" motor_prefix="fl" multiplier="-838" />
-        <xacro:control_motor_macro channel="3" motor_prefix="br" multiplier="-838" />
+        <xacro:macro_control_motor channel="0" motor_prefix="fr" multiplier="838" />
+        <xacro:macro_control_motor channel="1" motor_prefix="bl" multiplier="838" />
+        <xacro:macro_control_motor channel="2" motor_prefix="fl" multiplier="-838" />
+        <xacro:macro_control_motor channel="3" motor_prefix="br" multiplier="-838" />
       </plugin>
     </gazebo>
