Commit message: FPV Dron Model Added

File: urdf/fpv_drone.xacro (robot description, xacro)
@@ -1,4 +1,4 @@
 <?xml version="1.0"?>
-<robot name="test_fpv_drone" xmlns:xacro="http://www.ros.org/wiki/xacro">
+<robot name="fpv_drone" xmlns:xacro="http://www.ros.org/wiki/xacro">
   <xacro:arg name="package_name" default="fpv_drone" />
   <xacro:arg name="namespace" default="fpv_drone" />
@@ -9,4 +9,7 @@
   <xacro:arg name="rpy" default="0 0 0" />
   <xacro:arg name="xyz" default="0 0 0" />
+  <xacro:arg name="sitl" default="false" />
+  <xacro:arg name="gimbal" default="false" />
+  <xacro:arg name="instance" default="0" />
   <xacro:property name="package_name" value="$(arg package_name)" />
   <xacro:property name="namespace" value="$(arg namespace)" />
@@ -17,4 +20,7 @@
   <xacro:property name="rpy" value="$(arg rpy)" />
   <xacro:property name="xyz" value="$(arg xyz)" />
+  <xacro:property name="sitl" value="$(arg sitl)" />
+  <xacro:property name="gimbal" value="$(arg gimbal)" />
+  <xacro:property name="instance" value="$(arg instance)" />
   <xacro:property name="parent_link" value="${namespace}_footprint" />
   <xacro:include filename="$(find fpv_drone)/urdf/macro_fpv_drone.xacro" />
@@ -23,3 +29,17 @@
     parent_link="${parent_link}" rgb_base="${rgb_base}" rgb_cam="${rgb_cam}"
     rgb_ccw="${rgb_ccw}" rgb_cw="${rgb_cw}" rpy="${rpy}" xyz="${xyz}" />
+  <xacro:if value="${sitl}">
+    <xacro:include filename="$(find fpv_drone)/urdf/macro_sitl_core.xacro" />
+    <xacro:macro_sitl_core namespace="${namespace}" instance="${instance}" />
+  </xacro:if>
+  <xacro:if value="${gimbal}">
+    <xacro:include filename="$(find fpv_drone)/urdf/macro_gimbal_3d.xacro" />
+    <xacro:macro_gimbal_3d_macro package_name="${package_name}" namespace="${namespace}"
+      parent_link="${parent_link}" rgb="${rgb_cam}" instance="${instance}"
+      rpy="1.5707963267948966 0 1.5707963267948966" xyz="0 0 -0.03925" />
+    <xacro:if value="${sitl}">
+      <xacro:include filename="$(find fpv_drone)/urdf/macro_sitl_gimbal.xacro" />
+      <xacro:macro_sitl_gimbal namespace="${namespace}" />
+    </xacro:if>
+  </xacro:if>
 </robot>

File: urdf/macro_fpv_drone.xacro (robot description, xacro)
@@ -13,14 +13,14 @@
     <xacro:macro_fpv_motor package_name="${package_name}" namespace="${namespace}"
       parent_link="${namespace}_base_link"
-      prefix="fr" rgb="${rgb_ccw}" rpy="0 0 0" xyz="0.13541 -0.11532 0.01837" />
+      prefix="fr" rgb="${rgb_ccw}" rpy="0 0 0" xyz="0.1354 -0.11535 0.018367" />
     <xacro:macro_fpv_motor package_name="${package_name}" namespace="${namespace}"
       parent_link="${namespace}_base_link"
-      prefix="bl" rgb="${rgb_ccw}" rpy="0 0 0" xyz="-0.08106 0.11675 0.018367" />
+      prefix="bl" rgb="${rgb_ccw}" rpy="0 0 0" xyz="-0.081 0.1168 0.018367" />
     <xacro:macro_fpv_motor package_name="${package_name}" namespace="${namespace}"
       parent_link="${namespace}_base_link"
-      prefix="fl" rgb="${rgb_cw}" rpy="0 0 0" xyz="0.1353 0.11683 0.01837" />
+      prefix="fl" rgb="${rgb_cw}" rpy="0 0 0" xyz="0.1354 0.1168 0.018367" />
     <xacro:macro_fpv_motor package_name="${package_name}" namespace="${namespace}"
       parent_link="${namespace}_base_link"
-      prefix="br" rgb="${rgb_cw}" rpy="0 0 0" xyz="-0.08098 -0.11539 0.01837" />
+      prefix="br" rgb="${rgb_cw}" rpy="0 0 0" xyz="-0.081 -0.11535 0.018367" />
     <gazebo>
       <plugin

File: urdf/macro_gimbal_3d.xacro (robot description, xacro)
@@ -3,8 +3,8 @@
   <xacro:macro name="macro_gimbal_3d"
     params="package_name:='fpv_drone' namespace:='fpv_drone' parent_link:='fpv_drone_footprint' rgb:='0 1 1' instance:='0' rpy:='0 0 0' xyz:='0 0 0'">
+    <xacro:property name="namespace_gimbal" value="${namespace}_gimbal" />
+    <xacro:property name="STREAM_PORT" value="${5600 + int(instance) * 10}" />
     <xacro:property name="pi" value="3.141592653589793" />
     <xacro:property name="use_sim_time" value="true" />
-    <xacro:property name="namespace_gimbal" value="${namespace}_gimbal" />
-    <xacro:property name="STREAM_PORT" value="${5600 + int(instance) * 10}" />
     <link name="${namespace_gimbal}_base_link">
       <inertial>

File: urdf/macro_sitl_core.xacro (robot description, xacro)
@@ -47,5 +47,5 @@
       <xacro:macro_liftdrag_plugin motor_prefix="br" cp_vec="-0.042 -0.0727 0"
         fwd_vec="-0.866 0.5 0" />
-      <xacro:macro name="apply_joint_force_plugin_macro" params="motor_prefix">
+      <xacro:macro name="macro_apply_joint_force_plugin" params="motor_prefix">
         <plugin filename="gz-sim-apply-joint-force-system"
           name="gz::sim::systems::ApplyJointForce">
@@ -53,8 +53,8 @@
         </plugin>
       </xacro:macro>
-      <xacro:apply_joint_force_plugin_macro motor_prefix="fr" />
-      <xacro:apply_joint_force_plugin_macro motor_prefix="bl" />
-      <xacro:apply_joint_force_plugin_macro motor_prefix="fl" />
-      <xacro:apply_joint_force_plugin_macro motor_prefix="br" />
+      <xacro:macro_apply_joint_force_plugin motor_prefix="fr" />
+      <xacro:macro_apply_joint_force_plugin motor_prefix="bl" />
+      <xacro:macro_apply_joint_force_plugin motor_prefix="fl" />
+      <xacro:macro_apply_joint_force_plugin motor_prefix="br" />
       <plugin name="ArduPilotPlugin" filename="ArduPilotPlugin">
         <fdm_addr>127.0.0.1</fdm_addr>

File: urdf/test_fpv_ardupilot.xacro (robot description, xacro)
@@ -1,5 +1,4 @@
 <?xml version="1.0"?>
 <robot name="test_fpv_ardupilot" xmlns:xacro="http://www.ros.org/wiki/xacro">
-  <xacro:include filename="$(find fpv_drone)/urdf/macro_fpv_ardupilot.xacro" />
   <xacro:arg name="package_name" default="fpv_drone" />
   <xacro:arg name="namespace" default="fpv_drone" />
@@ -21,5 +20,5 @@
   <xacro:property name="instance" value="$(arg instance)" />
   <xacro:property name="parent_link" value="${namespace}_footprint" />
-  <xacro:property name="use_sim_time" value="true" />
+  <xacro:include filename="$(find fpv_drone)/urdf/macro_fpv_ardupilot.xacro" />
   <link name="${parent_link}" />
   <xacro:macro_fpv_ardupilot package_name="${package_name}" namespace="${namespace}"

File: urdf/test_fpv_base.xacro (robot description, xacro)
@@ -1,5 +1,4 @@
 <?xml version="1.0"?>
 <robot name="test_fpv_base" xmlns:xacro="http://www.ros.org/wiki/xacro">
-  <xacro:include filename="$(find fpv_drone)/urdf/macro_fpv_base.xacro" />
   <xacro:arg name="package_name" default="fpv_drone" />
   <xacro:arg name="namespace" default="fpv_drone" />
@@ -7,5 +6,5 @@
   <xacro:property name="namespace" value="$(arg namespace)" />
   <xacro:property name="parent_link" value="${namespace}_footprint" />
-  <xacro:property name="use_sim_time" value="true" />
+  <xacro:include filename="$(find fpv_drone)/urdf/macro_fpv_base.xacro" />
   <link name="${parent_link}">
     <inertial>

File: urdf/test_fpv_cam.xacro (robot description, xacro)
@@ -1,5 +1,4 @@
 <?xml version="1.0"?>
 <robot name="test_fpv_cam" xmlns:xacro="http://www.ros.org/wiki/xacro">
-  <xacro:include filename="$(find fpv_drone)/urdf/macro_fpv_cam.xacro" />
   <xacro:arg name="package_name" default="fpv_drone" />
   <xacro:arg name="namespace" default="fpv_drone" />
@@ -7,5 +6,5 @@
   <xacro:property name="namespace" value="$(arg namespace)" />
   <xacro:property name="parent_link" value="${namespace}_footprint" />
-  <xacro:property name="use_sim_time" value="true" />
+  <xacro:include filename="$(find fpv_drone)/urdf/macro_fpv_cam.xacro" />
   <link name="${parent_link}">
     <inertial>

File: urdf/test_fpv_motor.xacro (robot description, xacro)
@@ -1,5 +1,4 @@
 <?xml version="1.0"?>
 <robot name="test_fpv_motor" xmlns:xacro="http://www.ros.org/wiki/xacro">
-  <xacro:include filename="$(find fpv_drone)/urdf/macro_fpv_motor.xacro" />
   <xacro:arg name="package_name" default="fpv_drone" />
   <xacro:arg name="namespace" default="fpv_drone" />
@@ -7,5 +6,5 @@
   <xacro:property name="namespace" value="$(arg namespace)" />
   <xacro:property name="parent_link" value="${namespace}_footprint" />
-  <xacro:property name="use_sim_time" value="true" />
+  <xacro:include filename="$(find fpv_drone)/urdf/macro_fpv_motor.xacro" />
   <link name="${parent_link}">
     <inertial>

File: urdf/test_gimbal_3d.xacro (robot description, xacro)
@@ -1,5 +1,4 @@
 <?xml version="1.0"?>
 <robot name="test_gimbal_3d" xmlns:xacro="http://www.ros.org/wiki/xacro">
-  <xacro:include filename="$(find fpv_drone)/urdf/macro_gimbal_3d.xacro" />
   <xacro:arg name="package_name" default="fpv_drone" />
   <xacro:arg name="namespace" default="fpv_drone" />
@@ -7,5 +6,5 @@
   <xacro:property name="namespace" value="$(arg namespace)" />
   <xacro:property name="parent_link" value="${namespace}_footprint" />
-  <xacro:property name="use_sim_time" value="true" />
+  <xacro:include filename="$(find fpv_drone)/urdf/macro_gimbal_3d.xacro" />
   <link name="${parent_link}">
     <inertial>

Commit message: Rearrangements have been made

File: urdf/fpv_drone.xacro (robot description, xacro)
@@ -29,17 +29,13 @@
     parent_link="${parent_link}" rgb_base="${rgb_base}" rgb_cam="${rgb_cam}"
     rgb_ccw="${rgb_ccw}" rgb_cw="${rgb_cw}" rpy="${rpy}" xyz="${xyz}" />
+  <xacro:if value="${gimbal}">
+    <xacro:include filename="$(find fpv_drone)/urdf/macro_gimbal_3d.xacro" />
+    <xacro:macro_gimbal_3d package_name="${package_name}" namespace="${namespace}"
+      parent_link="${parent_link}" rgb="${rgb_cam}" instance="${instance}"
+      rpy="1.5707963267948966 0 1.5707963267948966" xyz="0 -0.01 -0.11775" />
+  </xacro:if>
   <xacro:if value="${sitl}">
     <xacro:include filename="$(find fpv_drone)/urdf/macro_sitl_core.xacro" />
-    <xacro:macro_sitl_core namespace="${namespace}" instance="${instance}" />
-  </xacro:if>
-  <xacro:if value="${gimbal}">
-    <xacro:include filename="$(find fpv_drone)/urdf/macro_gimbal_3d.xacro" />
-    <xacro:macro_gimbal_3d_macro package_name="${package_name}" namespace="${namespace}"
-      parent_link="${parent_link}" rgb="${rgb_cam}" instance="${instance}"
-      rpy="1.5707963267948966 0 1.5707963267948966" xyz="0 0 -0.03925" />
-    <xacro:if value="${sitl}">
-      <xacro:include filename="$(find fpv_drone)/urdf/macro_sitl_gimbal.xacro" />
-      <xacro:macro_sitl_gimbal namespace="${namespace}" />
-    </xacro:if>
+    <xacro:macro_sitl_core namespace="${namespace}" instance="${instance}" gimbal="${gimbal}" />
   </xacro:if>
 </robot>

File: urdf/macro_gimbal_3d.xacro (robot description, xacro)
@@ -7,4 +7,43 @@
     <xacro:property name="pi" value="3.141592653589793" />
     <xacro:property name="use_sim_time" value="true" />
+    <link name="${namespace_gimbal}_standoffs_link">
+      <inertial>
+        <mass value="0.01" />
+        <inertia ixx="0.00001" ixy="0" ixz="0" iyy="0.00001" iyz="0" izz="0.00001" />
+      </inertial>
+      <xacro:macro name="macro_standoffs_link" params="prefix size rpy xyz">
+        <visual name="${namespace_gimbal}_standoffs_visual_${prefix}">
+          <origin xyz="${xyz}" rpy="${rpy}" />
+          <geometry>
+            <box size="${size}" />
+          </geometry>
+          <material name="${namespace_gimbal}_material">
+            <color rgba="${rgb} 1" />
+          </material>
+        </visual>
+        <collision name="${namespace_gimbal}_standoffs_collision_${prefix}">
+          <origin xyz="${xyz}" rpy="${rpy}" />
+          <geometry>
+            <box size="${size}" />
+          </geometry>
+        </collision>
+      </xacro:macro>
+      <xacro:macro_standoffs_link prefix="fr" size="0.01 0.01 0.2"
+        rpy="0 0 0" xyz="0.12 -0.11 -0.11" />
+      <xacro:macro_standoffs_link prefix="fl" size="0.01 0.01 0.2"
+        rpy="0 0 0" xyz="-0.08 -0.11 -0.11" />
+      <xacro:macro_standoffs_link prefix="br" size="0.01 0.01 0.2"
+        rpy="0 0 0" xyz="0.12 0.11 -0.11" />
+      <xacro:macro_standoffs_link prefix="bl" size="0.01 0.01 0.2"
+        rpy="0 0 0" xyz="-0.08 0.11 -0.11" />
+    </link>
+    <joint name="${namespace_gimbal}_standoffs_joint" type="fixed">
+      <parent link="${parent_link}" />
+      <child link="${namespace_gimbal}_standoffs_link" />
+      <origin xyz="0 0 0" rpy="0 0 0" />
+      <axis xyz="0 0 1">
+        <limit lower="0" upper="0" effort="0" velocity="0" />
+      </axis>
+    </joint>
     <link name="${namespace_gimbal}_base_link">
       <inertial>

File: urdf/macro_sitl_core.xacro (robot description, xacro)
@@ -2,6 +2,9 @@
 <robot xmlns:xacro="http://www.ros.org/wiki/xacro">
   <xacro:macro name="macro_sitl_core"
-    params="namespace:='fpv_drone' instance:='0'">
+    params="namespace:='fpv_drone' instance:='0' gimbal:='false'">
     <xacro:property name="SITL_PORT" value="${9002 + int(instance) * 10}" />
+    <xacro:if value="${gimbal}">
+      <xacro:include filename="$(find fpv_drone)/urdf/macro_sitl_gimbal.xacro" />
+    </xacro:if>
     <gazebo>
       <xacro:macro name="macro_liftdrag_plugin" params="motor_prefix cp_vec fwd_vec">
@@ -89,5 +92,11 @@
         <xacro:macro_control_motor channel="2" motor_prefix="fl" multiplier="-838" />
         <xacro:macro_control_motor channel="3" motor_prefix="br" multiplier="-838" />
+        <xacro:if value="${gimbal}">
+          <xacro:macro_sitl_gimbal_sitl namespace="${namespace}" />
+        </xacro:if>
       </plugin>
+      <xacro:if value="${gimbal}">
+        <xacro:macro_sitl_gimbal_plugin namespace="${namespace}" />
+      </xacro:if>
     </gazebo>
   </xacro:macro>

File: urdf/macro_sitl_gimbal.xacro (robot description, xacro)
@@ -1,39 +1,37 @@
 <?xml version="1.0"?>
 <robot xmlns:xacro="http://www.ros.org/wiki/xacro">
-  <xacro:macro name="macro_sitl_gimbal"
-    params="namespace:='fpv_drone'">
-    <gazebo>
-      <plugin name="ArduPilotPlugin" filename="ArduPilotPlugin">
-        <xacro:macro name="macro_control_gimbal" params="channel prefix multiplier offset">
-          <control channel="${channel}">
-            <jointName>${namespace}_gimbal_${prefix}_joint</jointName>
-            <multiplier>${multiplier}</multiplier>
-            <offset>${offset}</offset>
-            <servo_min>1100</servo_min>
-            <servo_max>1900</servo_max>
-            <type>COMMAND</type>
-            <cmd_topic>${namespace}_gimbal_${prefix}_cmd</cmd_topic>
-            <p_gain>2</p_gain>
-          </control>
-        </xacro:macro>
-        <xacro:macro_control_gimbal channel="8" prefix="roll" multiplier="1.047197551196"
-          offset="-0.5" />
-        <xacro:macro_control_gimbal channel="9" prefix="pitch" multiplier="-3.14159265"
-          offset="-0.75" />
-        <xacro:macro_control_gimbal channel="10" prefix="yaw" multiplier="-5.5850536" offset="-0.5" />
+  <xacro:macro name="macro_sitl_gimbal_sitl" params="namespace:='fpv_drone'">
+    <xacro:macro name="macro_control_gimbal" params="channel prefix multiplier offset">
+      <control channel="${channel}">
+        <jointName>${namespace}_gimbal_${prefix}_joint</jointName>
+        <multiplier>${multiplier}</multiplier>
+        <offset>${offset}</offset>
+        <servo_min>1100</servo_min>
+        <servo_max>1900</servo_max>
+        <type>COMMAND</type>
+        <cmd_topic>/${namespace}_gimbal/${prefix}_cmd</cmd_topic>
+        <p_gain>2</p_gain>
+      </control>
+    </xacro:macro>
+    <xacro:macro_control_gimbal channel="8" prefix="roll" multiplier="1.047197551196"
+      offset="-0.5" />
+    <xacro:macro_control_gimbal channel="9" prefix="pitch" multiplier="-3.14159265"
+      offset="-0.75" />
+    <xacro:macro_control_gimbal channel="10" prefix="yaw" multiplier="-5.5850536"
+      offset="-0.5" />
+  </xacro:macro>
+  <xacro:macro name="macro_sitl_gimbal_plugin" params="namespace:='fpv_drone'">
+    <xacro:macro name="macro_joint_position_controller" params="prefix">
+      <plugin
+        filename="gz-sim-joint-position-controller-system"
+        name="gz::sim::systems::JointPositionController">
+        <joint>${namespace}_gimbal_${prefix}_joint</joint>
+        <topic>/${namespace}_gimbal/${prefix}_cmd</topic>
+        <p_gain>2</p_gain>
       </plugin>
-      <xacro:macro name="macro_joint_position_controller" params="prefix">
-        <plugin
-          filename="gz-sim-joint-position-controller-system"
-          name="gz::sim::systems::JointPositionController">
-          <joint>${namespace}_gimbal_${prefix}_joint</joint>
-          <topic>${namespace}_gimbal_${prefix}_cmd</topic>
-          <p_gain>2</p_gain>
-        </plugin>
-      </xacro:macro>
-      <xacro:macro_joint_position_controller prefix="roll" />
-      <xacro:macro_joint_position_controller prefix="pitch" />
-      <xacro:macro_joint_position_controller prefix="yaw" />
-    </gazebo>
+    </xacro:macro>
+    <xacro:macro_joint_position_controller prefix="roll" />
+    <xacro:macro_joint_position_controller prefix="pitch" />
+    <xacro:macro_joint_position_controller prefix="yaw" />
   </xacro:macro>
 </robot>
